File: bifocals-filter/lichen-bifocals-control-board/lichen-bifocals-control-board.kicad_sch (KiCad schematic)
At the start: 18 parts, among them J1 EURO_JACK, J2 EURO_JACK, J3 EURO_JACK, J4 EURO_JACK, J5 EURO_JACK, J6 EURO_JACK, J7 EURO_JACK, J8 EURO_JACK, J9 EURO_JACK

Commit message: v1.1 of Freddie and Bifocals hardware.
Other:
- title: Lichen Bifocals -> Lichen Bifocals Controls Board
Changed lines of the file:
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@@
   (paper "A4")
   (title_block
-    (title "Lichen Bifocals")
-    (date "2024-02-05")
-    (rev "1.0")
+    (title "Lichen Bifocals Controls Board")
+    (date "2024-08-30")
+    (rev "1.1")
     (company "Lichen Community Systems")
   )
@@
     (pin "9")
     (instances
-      (project "lichen-bifocals-board"
+      (project "lichen-bifocals-control-board"
         (path "/af83a72f-b7ee-4346-b6a2-eaa1468cc44d"
           (reference "H2") (unit 1)
@@
     (pin "1")
     (instances
-      (project "lichen-bifocals-board"
+      (project "lichen-bifocals-control-board"
         (path "/af83a72f-b7ee-4346-b6a2-eaa1468cc44d"
           (reference "#PWR018") (unit 1)
@@
     (pin "TIP")
     (instances
-      (project "lichen-bifocals-board"
+      (project "lichen-bifocals-control-board"
         (path "/af83a72f-b7ee-4346-b6a2-eaa1468cc44d"
           (reference "J6") (unit 1)
@@
     (pin "3")
     (instances
-      (project "lichen-bifocals-board"
+      (project "lichen-bifocals-control-board"
         (path "/af83a72f-b7ee-4346-b6a2-eaa1468cc44d"
           (reference "VR1") (unit 1)
@@
     (pin "1")
     (instances
-      (project "lichen-bifocals-board"
+      (project "lichen-bifocals-control-board"
         (path "/af83a72f-b7ee-4346-b6a2-eaa1468cc44d"
           (reference "#PWR026") (unit 1)
@@
     (pin "1")
     (instances
-      (project "lichen-bifocals-board"
+      (project "lichen-bifocals-control-board"
         (path "/af83a72f-b7ee-4346-b6a2-eaa1468cc44d"
           (reference "#PWR025") (unit 1)
@@
     (pin "1")
     (instances
-      (project "lichen-bifocals-board"
+      (project "lichen-bifocals-control-board"
         (path "/af83a72f-b7ee-4346-b6a2-eaa1468cc44d"
           (reference "#PWR027") (unit 1)
@@
     (pin "1")
     (instances
-      (project "lichen-bifocals-board"
+      (project "lichen-bifocals-control-board"
         (path "/af83a72f-b7ee-4346-b6a2-eaa1468cc44d"
           (reference "#PWR022") (unit 1)
@@
     (pin "1")
     (instances
-      (project "lichen-bifocals-board"
+      (project "lichen-bifocals-control-board"
         (path "/af83a72f-b7ee-4346-b6a2-eaa1468cc44d"
           (reference "#PWR029") (unit 1)
@@
     (pin "TIP")
     (instances
-      (project "lichen-bifocals-board"
+      (project "lichen-bifocals-control-board"
         (path "/af83a72f-b7ee-4346-b6a2-eaa1468cc44d"
           (reference "J4") (unit 1)
@@
     (pin "4")
     (instances
-      (project "lichen-bifocals-board"
+      (project "lichen-bifocals-control-board"
         (path "/af83a72f-b7ee-4346-b6a2-eaa1468cc44d"
           (reference "S1") (unit 1)
@@
     (pin "1")
     (instances
-      (project "lichen-bifocals-board"
+      (project "lichen-bifocals-control-board"
         (path "/af83a72f-b7ee-4346-b6a2-eaa1468cc44d"
           (reference "#PWR024") (unit 1)
@@
     (pin "TIP")
     (instances
-      (project "lichen-bifocals-board"
+      (project "lichen-bifocals-control-board"
         (path "/af83a72f-b7ee-4346-b6a2-eaa1468cc44d"
           (reference "J2") (unit 1)
@@
     (pin "1")
     (instances
-      (project "lichen-bifocals-board"
+      (project "lichen-bifocals-control-board"
         (path "/af83a72f-b7ee-4346-b6a2-eaa1468cc44d"
           (reference "#PWR015") (unit 1)
@@
     (pin "1")
     (instances
-      (project "lichen-bifocals-board"
+      (project "lichen-bifocals-control-board"
         (path "/af83a72f-b7ee-4346-b6a2-eaa1468cc44d"
           (reference "#PWR09") (unit 1)
@@
     (pin "1")
     (instances
-      (project "lichen-bifocals-board"
+      (project "lichen-bifocals-control-board"
         (path "/af83a72f-b7ee-4346-b6a2-eaa1468cc44d"
           (reference "#PWR014") (unit 1)
@@
     (pin "1")
     (instances
-      (project "lichen-bifocals-board"
+      (project "lichen-bifocals-control-board"
         (path "/af83a72f-b7ee-4346-b6a2-eaa1468cc44d"
           (reference "#PWR010") (unit 1)
@@
     (pin "1")
     (instances
-      (project "lichen-bifocals-board"
+      (project "lichen-bifocals-control-board"
         (path "/af83a72f-b7ee-4346-b6a2-eaa1468cc44d"
           (reference "#PWR019") (unit 1)
@@
     (pin "3")
     (instances
-      (project "lichen-bifocals-board"
+      (project "lichen-bifocals-control-board"
         (path "/af83a72f-b7ee-4346-b6a2-eaa1468cc44d"
           (reference "VR5") (unit 1)
@@
     (pin "3")
     (instances
-      (project "lichen-bifocals-board"
+      (project "lichen-bifocals-control-board"
         (path "/af83a72f-b7ee-4346-b6a2-eaa1468cc44d"
           (reference "VR4") (unit 1)
@@
     (pin "1")
     (instances
-      (project "lichen-bifocals-board"
+      (project "lichen-bifocals-control-board"
         (path "/af83a72f-b7ee-4346-b6a2-eaa1468cc44d"
           (reference "#PWR013") (unit 1)
@@
     (pin "1")
     (instances
-      (project "lichen-bifocals-board"
+      (project "lichen-bifocals-control-board"
         (path "/af83a72f-b7ee-4346-b6a2-eaa1468cc44d"
           (reference "#PWR016") (unit 1)
@@
     (pin "3")
     (instances
-      (project "lichen-bifocals-board"
+      (project "lichen-bifocals-control-board"
         (path "/af83a72f-b7ee-4346-b6a2-eaa1468cc44d"
           (reference "VR2") (unit 1)
@@
     (pin "TIP")
     (instances
-      (project "lichen-bifocals-board"
+      (project "lichen-bifocals-control-board"
         (path "/af83a72f-b7ee-4346-b6a2-eaa1468cc44d"
           (reference "J1") (unit 1)
@@
     (pin "1")
     (instances
-      (project "lichen-bifocals-board"
+      (project "lichen-bifocals-control-board"
         (path "/af83a72f-b7ee-4346-b6a2-eaa1468cc44d"
           (reference "#PWR020") (unit 1)
@@
     (pin "1")
     (instances
-      (project "lichen-bifocals-board"
+      (project "lichen-bifocals-control-board"
         (path "/af83a72f-b7ee-4346-b6a2-eaa1468cc44d"
           (reference "#PWR011") (unit 1)
@@
     (pin "TIP")
     (instances
-      (project "lichen-bifocals-board"
+      (project "lichen-bifocals-control-board"
         (path "/af83a72f-b7ee-4346-b6a2-eaa1468cc44d"
           (reference "J9") (unit 1)
@@
     (pin "3")
     (instances
-      (project "lichen-bifocals-board"
+      (project "lichen-bifocals-control-board"
         (path "/af83a72f-b7ee-4346-b6a2-eaa1468cc44d"
           (reference "VR3") (unit 1)
@@
         )
       )
-      (project "lichen-bifocals-board"
+      (project "lichen-bifocals-control-board"
         (path "/af83a72f-b7ee-4346-b6a2-eaa1468cc44d"
           (reference "#PWR04") (unit 1)
@@
     (pin "9")
     (instances
-      (project "lichen-bifocals-board"
+      (project "lichen-bifocals-control-board"
         (path "/af83a72f-b7ee-4346-b6a2-eaa1468cc44d"
           (reference "H1") (unit 1)
@@
     (pin "1")
     (instances
-      (project "lichen-bifocals-board"
+      (project "lichen-bifocals-control-board"
         (path "/af83a72f-b7ee-4346-b6a2-eaa1468cc44d"
           (reference "#PWR023") (unit 1)
@@
     (pin "1")
     (instances
-      (project "lichen-bifocals-board"
+      (project "lichen-bifocals-control-board"
         (path "/af83a72f-b7ee-4346-b6a2-eaa1468cc44d"
           (reference "#PWR017") (unit 1)
@@
     (pin "TIP")
     (instances
-      (project "lichen-bifocals-board"
+      (project "lichen-bifocals-control-board"
         (path "/af83a72f-b7ee-4346-b6a2-eaa1468cc44d"
           (reference "J5") (unit 1)
@@
     (pin "1")
     (instances
-      (project "lichen-bifocals-board"
+      (project "lichen-bifocals-control-board"
         (path "/af83a72f-b7ee-4346-b6a2-eaa1468cc44d"
           (reference "#PWR02") (unit 1)
@@
     (pin "TIP")
     (instances
-      (project "lichen-bifocals-board"
+      (project "lichen-bifocals-control-board"
         (path "/af83a72f-b7ee-4346-b6a2-eaa1468cc44d"
           (reference "J3") (unit 1)
@@
     (pin "1")
     (instances
-      (project "lichen-bifocals-board"
+      (project "lichen-bifocals-control-board"
         (path "/af83a72f-b7ee-4346-b6a2-eaa1468cc44d"
           (reference "#PWR03") (unit 1)
@@
     (pin "1")
     (instances
-      (project "lichen-bifocals-board"
+      (project "lichen-bifocals-control-board"
         (path "/af83a72f-b7ee-4346-b6a2-eaa1468cc44d"
           (reference "#PWR021") (unit 1)
@@
     (pin "1")
     (instances
-      (project "lichen-bifocals-board"
+      (project "lichen-bifocals-control-board"
         (path "/af83a72f-b7ee-4346-b6a2-eaa1468cc44d"
           (reference "#PWR012") (unit 1)
@@
     (pin "K")
     (instances
-      (project "lichen-bifocals-board"
+      (project "lichen-bifocals-control-board"
         (path "/af83a72f-b7ee-4346-b6a2-eaa1468cc44d"
           (reference "LED1") (unit 1)
@@
     (pin "TIP")
     (instances
-      (project "lichen-bifocals-board"
+      (project "lichen-bifocals-control-board"
         (path "/af83a72f-b7ee-4346-b6a2-eaa1468cc44d"
           (reference "J7") (unit 1)
@@
     (pin "TIP")
     (instances
-      (project "lichen-bifocals-board"
+      (project "lichen-bifocals-control-board"
         (path "/af83a72f-b7ee-4346-b6a2-eaa1468cc44d"
           (reference "J8") (unit 1)
@@
     (pin "1")
     (instances
-      (project "lichen-bifocals-board"
+      (project "lichen-bifocals-control-board"
         (path "/af83a72f-b7ee-4346-b6a2-eaa1468cc44d"
           (reference "#PWR01") (unit 1)
