File: bifocals-filter/lichen-bifocals-submodule-power-board/lichen-bifocals-submodule-power-board.kicad_sch (KiCad schematic)
At the start: 4 parts

Commit message: v1.1 of Freddie and Bifocals hardware.
Other:
- company: (none) -> Lichen Community Systems
- title: (none) -> Lichen Bifocals Submodule/Power Board
Changed lines of the file:
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@@
 (kicad_sch (version 20230121) (generator eeschema)
   (paper "A4")
+  (title_block
+    (title "Lichen Bifocals Submodule/Power Board")
+    (date "2024-08-30")
+    (rev "1.1")
+    (company "Lichen Community Systems")
+  )
   (no_connect (at 57.15 77.47))
   (no_connect (at 102.87 105.41))
