File: bifocals-filter/lichen-bifocals-submodule-power-board/lichen-bifocals-submodule-power-board.kicad_pcb (KiCad board)
At the start: 2 copper layers, 40.3 x 108 mm, 4 parts

Commit message: Updates Patch SM boards to non-exploding footprint.
Parts:
- MCU1: value ES_DAISY_PATCH_SM_REV1 -> Daisy Patch Submodule; footprint ES_Daisy_Patch_SM_FB_Rev1:ES_DAISY_PATCH_SM_REV1 -> Lichen:Daisy_Patch_Submodule
Changed lines of the file:
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@@
   (net 39 "unconnected-(MCU1-USB_DM-PadA8)")
   (net 40 "+12V")
-  (footprint "ES_Daisy_Patch_SM_FB_Rev1:ES_DAISY_PATCH_SM_REV1" (layer "F.Cu")
+  (footprint "Lichen:Daisy_Patch_Submodule" (layer "F.Cu")
     (at 120.29 150.813 90)
     (property "Sheetfile" "lichen-bifocals-submodule-power-board.kicad_sch")
@@
         (effects (font (size 1.27 1.27) (thickness 0.15)))
     )
-    (fp_text value "ES_DAISY_PATCH_SM_REV1" (at 0 0 90) (layer "B.SilkS")
+    (fp_text value "Daisy Patch Submodule" (at 32.393 -0.12) (layer "B.SilkS")
         (effects (font (size 1.27 1.27) (thickness 0.15)) (justify mirror))
     )

Commit message: v1.1 of Freddie and Bifocals hardware.
Parts:
- added MH1: MountingHole_2.2mm_M2, MountingHole:MountingHole_2.2mm_M2, F.Cu at (113.2, 203.1)
- added MH2: MountingHole_2.2mm_M2, MountingHole:MountingHole_2.2mm_M2, F.Cu at (127.1, 203.1)
Other:
- board text added: "August 2024"
- board text added: "Lichen Community Systems Bifocals v1.1"
- board text removed: "February 2024"
- board text removed: "Lichen Community Systems Bifocals v1.0"
