File: bifocals-filter/lichen-bifocals-panel/lichen-bifocals-panel.kicad_pcb (KiCad board)
At the start: 2 copper layers, 40.3 x 128.5 mm, 20 parts

Commit message: v1.1 of Freddie and Bifocals hardware.
Other:
- board text added: "August 2024"
- board text added: "Lichen Bifocals v1.1"
- board text removed: "February 2024"
- board text removed: "Lichen Bifocals v1.0"
