File: lichen-medium/lichen-medium-board/lichen-dev-module.kicad_pcb (KiCad board)
At the start: 2 copper layers, 68.6 x 108.2 mm, 22 parts, among them J1 Eurorack_Mono_Jack, J10 Eurorack_Mono_Jack, J11 Eurorack_Mono_Jack, J2 Eurorack_Mono_Jack, J3 Eurorack_Mono_Jack, J4 Eurorack_Mono_Jack, J5 Eurorack_Mono_Jack, J6 Eurorack_Mono_Jack, J7 Eurorack_Mono_Jack, J8 Eurorack_Mono_Jack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

Commit message: Updates Patch SM boards to non-exploding footprint.
Parts:
- MCU1: value ES_DAISY_PATCH_SM_REV1 -> Daisy Patch Submodule; footprint ES_Daisy_Patch_SM_FB_Rev1:ES_DAISY_PATCH_SM_REV1 -> Lichen:Daisy_Patch_Submodule
Other:
- board text added: "Lichen Community Systems Medium v1.3"
- board text added: "May 2024"
- board text removed: "Lichen Community Systems Medium v1.2"
- board text removed: "March 2024"
