File: lichen-passive-mutes/lichen-passive-mutes-board/lichen-passive-mutes-board.kicad_pcb (KiCad board)
At the start: 2 copper layers, 9.3 x 108 mm, 9 parts, among them J1 Eurorack_Mono_Jack, J2 Eurorack_Mono_Jack, J3 Eurorack_Mono_Jack, J4 Eurorack_Mono_Jack, J5 Eurorack_Mono_Jack, J6 Eurorack_Mono_Jack, SW1 SW_SPDT, SW2 SW_SPDT, SW3 SW_SPDT

Commit message: Fixes connections between jacks and switches on Lichen Sw. Now the panel is laid out so channels 1-3 are laid out sequentially.
Connections:
- SW1 pad 1: Net-(J3-Tip) -> Net-(J1-Tip)
- SW1 pad 2: Net-(J6-Tip) -> Net-(J4-Tip)
- SW3 pad 1: Net-(J1-Tip) -> Net-(J3-Tip)
- SW3 pad 2: Net-(J4-Tip) -> Net-(J6-Tip)
Routing:
- net Net-(J4-Tip): track 57.6 -> 35.1 mm
- net Net-(J1-Tip): track 105.8 -> 84.1 mm
- net Net-(J6-Tip): track 8.00 -> 29.5 mm
- net Net-(J3-Tip): track 58.1 -> 78.8 mm
- net Net-(J5-Tip): track 42.6 -> 44.5 mm
Other:
- board text added: "Cntrls."
- board text removed: "Components, this side."

Commit message: Updates Lichen component library and most module prototypes.
Other:
- board text added: "9.2024"
- board text added: "Lichen Sw v1.1, Copyright 2024 Colin Clark"
- board text removed: "Feb 2024"
- board text removed: "Lichen Sw v1.0, Copyright 2024 Colin Clark"
