File: lichen-four/lichen-four-board/lichen-four-board.kicad_pcb (KiCad board)
At the start: 2 copper layers, 58.1 x 108 mm, 39 parts, among them J1 Eurorack_Mono_Jack, J10 Eurorack_Mono_Jack, J11 Eurorack_Mono_Jack, J12 Eurorack_Mono_Jack, J13 Eurorack_Mono_Jack, J14 Eurorack_Mono_Jack, J2 Eurorack_Mono_Jack, J3 Eurorack_Mono_Jack, J4 Eurorack_Mono_Jack, J5 Eurorack_Mono_Jack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

Commit message: Scales Lichen Four CV outputs to -8V to 8V to match audio outputs.
Parts:
- R10, R5: value 820R -> 330R
- R2, R7: value 13k -> 22K
- R4, R9: value 5K -> 15K
Other:
- board text added: "Lichen Community Systems Four v1.1"
- board text added: "November 2024"
- board text removed: "Lichen Community Systems Four v1.0"
- board text removed: "September 2024"
