File: lichen-four/lichen-four-board/lichen-four-board.kicad_sch (KiCad schematic)
At the start: 39 parts, among them J1 Eurorack_Mono_Jack, J10 Eurorack_Mono_Jack, J11 Eurorack_Mono_Jack, J12 Eurorack_Mono_Jack, J13 Eurorack_Mono_Jack, J14 Eurorack_Mono_Jack, J2 Eurorack_Mono_Jack, J3 Eurorack_Mono_Jack, J4 Eurorack_Mono_Jack, J5 Eurorack_Mono_Jack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

Commit message: Scales Lichen Four CV outputs to -8V to 8V to match audio outputs.
Parts:
- R10, R5: value 820R_0603 -> 330R_0603; Display 820R -> 330R; LCSC C23253 -> C23410; Part Number 0603WAF8200T5E -> 0603WAF330LT5E; Specifications 820R, 1%, 1/10W, 0603 -> 330R, 1%, 1/10W, 0603
- R2, R7: value 13k_0603 -> 22k_0603; Display 13k -> 22k; LCSC C22797 -> C31850; Part Number 0603WAF1302T5E -> 0603WAF2202T5E; Specifications 13K, 1%, 1/10W, 0603 -> 22K, 1%, 1/10W, 0603
- R4: value 4.99K_0603 -> 15K_0603; Display 4.99k -> 15K; LCSC C23046 -> C22809; Part Number 0603WAF4991T5E -> 0603WAF1502T5E; Specifications 4.99K, 1%, 1/10W, 0603 -> 15K, 1%, 1/10W, 0603
- R9: value 5K_0603 -> 15K_0603; Display 4.99k -> 15k; LCSC C23046 -> C22809; Part Number 0603WAF4991T5E -> 0603WAF1502T5E; Specifications 4.99K, 1%, 1/10W, 0603 -> 15K, 1%, 1/10W, 0603
Changed lines of the file:
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@@
       (effects (font (size 1.27 1.27)))
     )
-    (property "Value" "5K_0603" (at 246.38 86.36 90)
+    (property "Value" "15K_0603" (at 246.38 86.36 90)
       (effects (font (size 1.27 1.27)) hide)
     )
@@
       (effects (font (size 1.27 1.27)) hide)
     )
-    (property "Specifications" "4.99K, 1%, 1/10W, 0603" (at 254.254 86.36 0)
+    (property "Specifications" "15K, 1%, 1/10W, 0603" (at 254.254 86.36 0)
       (effects (font (size 1.27 1.27)) (justify left) hide)
     )
@@
       (effects (font (size 1.27 1.27)) (justify left) hide)
     )
-    (property "Part Number" "0603WAF4991T5E" (at 257.302 86.36 0)
-      (effects (font (size 1.27 1.27)) (justify left) hide)
-    )
-    (property "Display" "4.99k" (at 246.38 80.01 90)
-      (effects (font (size 1.27 1.27)))
-    )
-    (property "LCSC" "C23046" (at 246.38 80.01 90)
+    (property "Part Number" "0603WAF1502T5E" (at 257.302 86.36 0)
+      (effects (font (size 1.27 1.27)) (justify left) hide)
+    )
+    (property "Display" "15k" (at 246.38 80.01 90)
+      (effects (font (size 1.27 1.27)))
+    )
+    (property "LCSC" "C22809" (at 246.38 80.01 90)
       (effects (font (size 1.27 1.27)) hide)
     )
@@
       (effects (font (size 1.27 1.27)) (justify left))
     )
-    (property "Value" "13k_0603" (at 238.76 88.9 90)
+    (property "Value" "22k_0603" (at 238.76 88.9 90)
       (effects (font (size 1.27 1.27)) hide)
     )
@@
       (effects (font (size 1.27 1.27)) hide)
     )
-    (property "Specifications" "13K, 1%, 1/10W, 0603" (at 238.76 96.774 0)
+    (property "Specifications" "22K, 1%, 1/10W, 0603" (at 238.76 96.774 0)
       (effects (font (size 1.27 1.27)) (justify left) hide)
     )
@@
       (effects (font (size 1.27 1.27)) (justify left) hide)
     )
-    (property "Part Number" "0603WAF1302T5E" (at 238.76 99.822 0)
-      (effects (font (size 1.27 1.27)) (justify left) hide)
-    )
-    (property "Display" "13k" (at 243.84 90.17 0)
-      (effects (font (size 1.27 1.27)) (justify left))
-    )
-    (property "LCSC" "C22797" (at 241.3 88.9 0)
+    (property "Part Number" "0603WAF2202T5E" (at 238.76 99.822 0)
+      (effects (font (size 1.27 1.27)) (justify left) hide)
+    )
+    (property "Display" "22k" (at 243.84 90.17 0)
+      (effects (font (size 1.27 1.27)) (justify left))
+    )
+    (property "LCSC" "C31850" (at 241.3 88.9 0)
       (effects (font (size 1.27 1.27)) hide)
     )
@@
       (effects (font (size 1.27 1.27)))
     )
-    (property "Value" "820R_0603" (at 215.9 57.15 90)
+    (property "Value" "330R_0603" (at 215.9 57.15 90)
       (effects (font (size 1.27 1.27)) hide)
     )
@@
       (effects (font (size 1.27 1.27)) hide)
     )
-    (property "Specifications" "820R, 1%, 1/10W, 0603" (at 223.774 57.15 0)
+    (property "Specifications" "330R, 1%, 1/10W, 0603" (at 223.774 57.15 0)
       (effects (font (size 1.27 1.27)) (justify left) hide)
     )
@@
       (effects (font (size 1.27 1.27)) (justify left) hide)
     )
-    (property "Part Number" "0603WAF8200T5E" (at 226.822 57.15 0)
-      (effects (font (size 1.27 1.27)) (justify left) hide)
-    )
-    (property "Display" "820R" (at 215.9 50.8 90)
-      (effects (font (size 1.27 1.27)))
-    )
-    (property "LCSC" "C23253" (at 231.14 54.61 0)
+    (property "Part Number" "0603WAF330LT5E" (at 226.822 57.15 0)
+      (effects (font (size 1.27 1.27)) (justify left) hide)
+    )
+    (property "Display" "330R" (at 215.9 50.8 90)
+      (effects (font (size 1.27 1.27)))
+    )
+    (property "LCSC" "C23410" (at 231.14 54.61 0)
       (effects (font (size 1.27 1.27)) hide)
     )
@@
       (effects (font (size 1.27 1.27)) (justify left))
     )
-    (property "Value" "13k_0603" (at 200.66 59.69 90)
+    (property "Value" "22k_0603" (at 200.66 59.69 90)
       (effects (font (size 1.27 1.27)) hide)
     )
@@
       (effects (font (size 1.27 1.27)) hide)
     )
-    (property "Specifications" "13K, 1%, 1/10W, 0603" (at 200.66 67.564 0)
+    (property "Specifications" "22K, 1%, 1/10W, 0603" (at 200.66 67.564 0)
       (effects (font (size 1.27 1.27)) (justify left) hide)
     )
@@
       (effects (font (size 1.27 1.27)) (justify left) hide)
     )
-    (property "Part Number" "0603WAF1302T5E" (at 200.66 70.612 0)
-      (effects (font (size 1.27 1.27)) (justify left) hide)
-    )
-    (property "Display" "13k" (at 205.74 60.96 0)
-      (effects (font (size 1.27 1.27)) (justify left))
-    )
-    (property "LCSC" "C22797" (at 203.2 59.69 0)
+    (property "Part Number" "0603WAF2202T5E" (at 200.66 70.612 0)
+      (effects (font (size 1.27 1.27)) (justify left) hide)
+    )
+    (property "Display" "22k" (at 205.74 60.96 0)
+      (effects (font (size 1.27 1.27)) (justify left))
+    )
+    (property "LCSC" "C31850" (at 203.2 59.69 0)
       (effects (font (size 1.27 1.27)) hide)
     )
@@
       (effects (font (size 1.27 1.27)))
     )
-    (property "Value" "4.99K_0603" (at 208.28 57.15 90)
+    (property "Value" "15K_0603" (at 208.28 57.15 90)
       (effects (font (size 1.27 1.27)) hide)
     )
@@
       (effects (font (size 1.27 1.27)) hide)
     )
-    (property "Specifications" "4.99K, 1%, 1/10W, 0603" (at 216.154 57.15 0)
+    (property "Specifications" "15K, 1%, 1/10W, 0603" (at 216.154 57.15 0)
       (effects (font (size 1.27 1.27)) (justify left) hide)
     )
@@
       (effects (font (size 1.27 1.27)) (justify left) hide)
     )
-    (property "Part Number" "0603WAF4991T5E" (at 219.202 57.15 0)
-      (effects (font (size 1.27 1.27)) (justify left) hide)
-    )
-    (property "Display" "4.99k" (at 208.28 50.8 90)
-      (effects (font (size 1.27 1.27)))
-    )
-    (property "LCSC" "C23046" (at 208.28 50.8 90)
+    (property "Part Number" "0603WAF1502T5E" (at 219.202 57.15 0)
+      (effects (font (size 1.27 1.27)) (justify left) hide)
+    )
+    (property "Display" "15K" (at 208.28 50.8 90)
+      (effects (font (size 1.27 1.27)))
+    )
+    (property "LCSC" "C22809" (at 208.28 50.8 90)
       (effects (font (size 1.27 1.27)) hide)
     )
@@
       (effects (font (size 1.27 1.27)))
     )
-    (property "Value" "820R_0603" (at 254 86.36 90)
+    (property "Value" "330R_0603" (at 254 86.36 90)
       (effects (font (size 1.27 1.27)) hide)
     )
@@
       (effects (font (size 1.27 1.27)) hide)
     )
-    (property "Specifications" "820R, 1%, 1/10W, 0603" (at 261.874 86.36 0)
+    (property "Specifications" "330R, 1%, 1/10W, 0603" (at 261.874 86.36 0)
       (effects (font (size 1.27 1.27)) (justify left) hide)
     )
@@
       (effects (font (size 1.27 1.27)) (justify left) hide)
     )
-    (property "Part Number" "0603WAF8200T5E" (at 264.922 86.36 0)
-      (effects (font (size 1.27 1.27)) (justify left) hide)
-    )
-    (property "Display" "820R" (at 254 80.01 90)
-      (effects (font (size 1.27 1.27)))
-    )
-    (property "LCSC" "C23253" (at 269.24 83.82 0)
-      (effects (font (size 1.27 1.27)) hide)
-    )
+    (property "Part Number" "0603WAF330LT5E" (at 264.922 86.36 0)
+      (effects (font (size 1.27 1.27)) (justify left) hide)
+    )
+    (property "Display" "330R" (at 254 80.01 90)
+      (effects (font (size 1.27 1.27)))
+    )
+    (property "LCSC" "C23410" (at 269.24 83.82 0)
+      (effects (font (size 1.27 1.27)) hide)
+    )

Commit message: Adds design blocks.
Parts:
- PWR1: footprint winterbloom:Eurorack_Power_2x5_Shrouded_Lock -> Lichen:Eurorack_Power_SMD
