File: active-vactrol-vca/active-vactrol-vca-board/Left_Gate.kicad_sch (KiCad schematic)
At the start: 17 parts, among them J1 Thonkiconn_Mono_Audio_Jack, J2 Thonkiconn_Mono_Audio_Jack, J3 Thonkiconn_Mono_Audio_Jack, U1 TL072, U2 TL072, U5 NSL-32R3 60R@20mA

Commit message: Updates Lichen symbols and footprints. Fixes to Crustose and Vactrol VCA. Adds 3D model of the RP2350 dual USB board.
Parts:
- C4: now left out of the parts list
- J1, J2, J3: footprint Lichen:Audio_Jack_Thonkiconn_Mono -> Lichen:Audio_Jack_Thonkiconn_Mono_Left_Overhang; now left out of the parts list
- R1, R2, R3, R4, R5: value 100k -> 100k_0603; JLCPCB ID C25803 -> (none); LCSC (none) -> C25803
- R20, R8: value 10k_0603 -> 100k_0603; JLCPCB ID C25803 -> (none); LCSC (none) -> C25803
- R9: value 10k_0603 -> 1k_0603; JLCPCB ID C25804 -> (none)
- RV1: symbol Lichen:Potentiometer -> Lichen:R_Potentiometer; now left out of the parts list
- U5: symbol Isolator:NSL-32 -> Lichen:NSL-32
Connections:
- net GND: now also RV1.1, U5.1 (A); no longer RV1.3, U5.2 (K)
- net L_CV_ATTENUATED: now also U5.2 (K); no longer U5.1 (A)
- net L_CV_BUFFERED: now also RV1.3; no longer RV1.1
Other:
- note added: "Vactrol LED connection is backwards, because the CV has been inverted."
Changed lines of the file:
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@@
 		)
 	)
+	(text "Vactrol LED connection is backwards,\nbecause the CV has been inverted."
+		(exclude_from_sim no)
+		(at 168.148 90.17 0)
+		(effects
+			(font
+				(size 1.27 1.27)
+			)
+		)
+	)
 	(text "CV attuenuator"
 		(exclude_from_sim no)
@@
 	(wire
 		(pts
-			(xy 142.24 95.25) (xy 142.24 99.06)
-		)
-		(stroke
-			(width 0)
-			(type default)
-		)
-	)
-	(wire
-		(pts
 			(xy 82.55 127) (xy 83.82 127)
 		)
@@
 	(wire
 		(pts
-			(xy 153.67 82.55) (xy 153.67 99.06)
+			(xy 148.59 82.55) (xy 148.59 99.06)
 		)
 		(stroke
@@
 	(wire
 		(pts
-			(xy 148.59 95.25) (xy 142.24 95.25)
+			(xy 153.67 93.98) (xy 160.02 93.98)
 		)
 		(stroke
@@
 	(wire
 		(pts
-			(xy 119.38 82.55) (xy 153.67 82.55)
+			(xy 119.38 82.55) (xy 148.59 82.55)
 		)
 		(stroke
@@
 	(wire
 		(pts
-			(xy 148.59 99.06) (xy 148.59 95.25)
+			(xy 153.67 99.06) (xy 153.67 93.98)
 		)
 		(stroke
@@
 			)
 		)
-		(property "Value" "100k"
+		(property "Value" "100k_0603"
 			(at 91.44 63.5 90)
 			(effects
@@
 			)
 		)
-		(property "JLCPCB ID" "C25803"
+		(property "LCSC" "C25803"
 			(at 106.68 67.31 0)
 			(effects
@@
 		(unit 1)
 		(exclude_from_sim no)
-		(in_bom yes)
+		(in_bom no)
 		(on_board yes)
 		(dnp no)
@@
 			)
 		)
-		(property "Value" "10k_0603"
+		(property "Value" "1k_0603"
 			(at 223.52 119.38 90)
 			(effects
@@
 			)
 		)
-		(property "JLCPCB ID" "C25804"
-			(at 238.76 123.19 0)
-			(effects
-				(font
-					(size 1.27 1.27)
-				)
-				(hide yes)
-			)
-		)
 		(property "LCSC" "C21190"
 			(at 241.554 123.19 0)
@@
 			)
 		)
-		(property "Value" "100k"
+		(property "Value" "100k_0603"
 			(at 73.66 124.46 90)
 			(effects
@@
 			)
 		)
-		(property "JLCPCB ID" "C25803"
+		(property "LCSC" "C25803"
 			(at 88.9 120.65 0)
 			(effects
@@
 			)
 		)
-		(property "Value" "100k"
+		(property "Value" "100k_0603"
 			(at 33.02 62.23 90)
 			(effects
@@
 			)
 		)
-		(property "JLCPCB ID" "C25803"
+		(property "LCSC" "C25803"
 			(at 36.83 77.47 0)
 			(effects
@@
 			)
 		)
-		(property "LCSC" "C6961"
+		(property "Manufacturer" "STMicroelectronics"
 			(at 181.61 119.38 0)
 			(effects
@@
 			)
 		)
-		(property "Manufacturer" "STMicroelectronics"
+		(property "Part Number" "TL072CDT"
 			(at 181.61 119.38 0)
 			(effects
@@
 			)
 		)
-		(property "Part Number" "TL072CDT"
+		(property "LCSC" "C6961"
 			(at 181.61 119.38 0)
 			(effects
@@
 		(unit 1)
 		(exclude_from_sim no)
-		(in_bom yes)
+		(in_bom no)
 		(on_board yes)
 		(dnp no)
@@
 			)
 		)
-		(property "Footprint" "Lichen:Audio_Jack_Thonkiconn_Mono"
+		(property "Footprint" "Lichen:Audio_Jack_Thonkiconn_Mono_Left_Overhang"
 			(at 264.414 106.172 0)
 			(effects
@@
 			)
 		)
-		(property "Value" "10k_0603"
+		(property "Value" "100k_0603"
 			(at 195.58 121.92 90)
 			(effects
@@
 			)
 		)
-		(property "JLCPCB ID" "C25803"
+		(property "LCSC" "C25803"
 			(at 210.82 118.11 0)
 			(effects
@@
 		(unit 1)
 		(exclude_from_sim no)
-		(in_bom yes)
+		(in_bom no)
 		(on_board yes)
 		(dnp no)
@@
 			)
 		)
-		(property "Footprint" "Lichen:Audio_Jack_Thonkiconn_Mono"
+		(property "Footprint" "Lichen:Audio_Jack_Thonkiconn_Mono_Left_Overhang"
 			(at 31.496 56.642 0)
 			(effects
@@
 			)
 		)
-		(property "Value" "100k"
+		(property "Value" "100k_0603"
 			(at 74.93 74.93 90)
 			(effects
@@
 			)
 		)
-		(property "JLCPCB ID" "C25803"
+		(property "LCSC" "C25803"
 			(at 90.17 71.12 0)
 			(effects
@@
 			)
 		)
-		(property "Value" "100k"
+		(property "Value" "100k_0603"
 			(at 91.44 113.03 90)
 			(effects
@@
 			)
 		)
-		(property "JLCPCB ID" "C25803"
+		(property "LCSC" "C25803"
 			(at 106.68 116.84 0)
 			(effects
@@
 			)
 		)
-		(property "Value" "10k_0603"
+		(property "Value" "100k_0603"
 			(at 217.17 106.68 90)
 			(effects
@@
 			)
 		)
-		(property "JLCPCB ID" "C25803"
+		(property "LCSC" "C25803"
 			(at 232.41 110.49 0)
 			(effects
@@
 			)
 		)
-		(property "LCSC" "C6961"
+		(property "Manufacturer" "STMicroelectronics"
 			(at 91.44 124.46 0)
 			(effects
@@
 			)
 		)
-		(property "Manufacturer" "STMicroelectronics"
+		(property "Part Number" "TL072CDT"
 			(at 91.44 124.46 0)
 			(effects
@@
 			)
 		)
-		(property "Part Number" "TL072CDT"
+		(property "LCSC" "C6961"
 			(at 91.44 124.46 0)
 			(effects
@@
 	)
 	(symbol
-		(lib_id "Isolator:NSL-32")
+		(lib_id "Lichen:NSL-32")
 		(at 151.13 106.68 270)
 		(unit 1)
@@
 			)
 		)
-		(property "LCSC" "C6961"
+		(property "Manufacturer" "STMicroelectronics"
 			(at 91.44 74.93 0)
 			(effects
@@
 			)
 		)
-		(property "Manufacturer" "STMicroelectronics"
+		(property "Part Number" "TL072CDT"
 			(at 91.44 74.93 0)
 			(effects
@@
 			)
 		)
-		(property "Part Number" "TL072CDT"
+		(property "LCSC" "C6961"
 			(at 91.44 74.93 0)
 			(effects
@@
 	(symbol
 		(lib_id "power:GND")
-		(at 142.24 99.06 0)
+		(at 160.02 93.98 0)
+		(mirror y)
 		(unit 1)
 		(exclude_from_sim no)
@@
 		(fields_autoplaced yes)
 		(property "Reference" "#PWR020"
-			(at 142.24 105.41 0)
+			(at 160.02 100.33 0)
 			(effects
 				(font
@@
 		)
 		(property "Value" "GND"
-			(at 142.24 104.14 0)
+			(at 160.02 99.06 0)
 			(effects
 				(font
@@
 		)
 		(property "Footprint" ""
-			(at 142.24 99.06 0)
+			(at 160.02 93.98 0)
 			(effects
 				(font
@@
 		)
 		(property "Datasheet" ""
-			(at 142.24 99.06 0)
+			(at 160.02 93.98 0)
 			(effects
 				(font
@@
 		)
 		(property "Description" "Power symbol creates a global label with name \"GND\" , ground"
-			(at 142.24 99.06 0)
+			(at 160.02 93.98 0)
 			(effects
 				(font
@@
 	)
 	(symbol
-		(lib_id "Lichen:Potentiometer")
+		(lib_id "Lichen:R_Potentiometer")
 		(at 115.57 82.55 0)
+		(mirror x)
 		(unit 1)
 		(exclude_from_sim no)
-		(in_bom yes)
+		(in_bom no)
 		(on_board yes)
 		(dnp no)
-		(fields_autoplaced yes)
 		(property "Reference" "RV1"
-			(at 113.03 81.2799 0)
+			(at 113.03 83.8201 0)
 			(effects
 				(font
@@
 		)
 		(property "Value" "B10K"
-			(at 113.03 83.8199 0)
+			(at 113.03 81.2801 0)
 			(effects
 				(font
@@
 		)
 		(property "Footprint" "Lichen:Potentiometer_Alpha_RD901_Eurorack"
-			(at 115.57 100.838 0)
+			(at 115.57 64.262 0)
 			(effects
 				(font
@@
 		)
 		(property "Datasheet" "https://www.thonk.co.uk/wp-content/uploads/2017/12/Alpha-9mm-Vertical-T18-RD901F-40-15K-B50K-0057.pdf"
-			(at 116.586 98.552 0)
+			(at 116.586 66.548 0)
 			(effects
 				(font
@@
 		)
 		(property "Description" "Alpha RD901 Vertical Snap-In Potentiometer"
-			(at 115.316 70.104 0)
+			(at 115.316 94.996 0)
 			(effects
 				(font
@@
 		)
 		(property "Part Number" "RD901F-40"
-			(at 115.57 96.52 0)
+			(at 115.57 68.58 0)
 			(effects
 				(font
@@
 		)
 		(property "Manufacturer" "Taiwan Alpha Electronic"
-			(at 116.078 94.488 0)
+			(at 116.078 70.612 0)
 			(effects
 				(font
@@
 		(unit 1)
 		(exclude_from_sim no)
-		(in_bom yes)
+		(in_bom no)
 		(on_board yes)
 		(dnp no)
@@
 			)
 		)
-		(property "Footprint" "Lichen:Audio_Jack_Thonkiconn_Mono"
+		(property "Footprint" "Lichen:Audio_Jack_Thonkiconn_Mono_Left_Overhang"
 			(at 31.496 106.172 0)
 			(effects
