File: active-vactrol-vca/active-vactrol-vca-board/Right_Gate.kicad_sch (KiCad schematic)
At the start: 16 parts, among them J4 Thonkiconn_Mono_Audio_Jack, J5 Thonkiconn_Mono_Audio_Jack, J6 Thonkiconn_Mono_Audio_Jack, U3 TL072, U4 TL072, U6 NSL-32R3 60R@20mA

Commit message: Updates Lichen symbols and footprints. Fixes to Crustose and Vactrol VCA. Adds 3D model of the RP2350 dual USB board.
Parts:
- C7: now left out of the parts list
- J4, J5, J6: footprint Lichen:Audio_Jack_Thonkiconn_Mono -> Lichen:Audio_Jack_Thonkiconn_Mono_Right_Overhang; now left out of the parts list
- R10, R11, R12, R13: value 100k -> 100k_0603; JLCPCB ID C25803 -> (none); LCSC (none) -> C25803
- R17, R19: value 10k_0603 -> 100k_0603; JLCPCB ID C25803 -> (none); LCSC (none) -> C25803
- R18: value 10k_0603 -> 1k_0603; JLCPCB ID C25804 -> (none)
- RV2: symbol Lichen:Potentiometer -> Lichen:R_Potentiometer; now left out of the parts list
- U6: symbol Isolator:NSL-32 -> Lichen:NSL-32; now left out of the parts list
Connections:
- net GND: now also RV2.1, U6.1 (A); no longer RV2.3, U6.2 (K)
- net R_CV_ATTENUATED: now also U6.2 (K); no longer U6.1 (A)
- net R_CV_BUFFERED: now also RV2.3; no longer RV2.1
Other:
- note removed: "TODO: Change to 0.1uF or 0.15uF cap due to reduced current from the 10k pot"
Changed lines of the file:
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@@
-		)
-	)
-	(text "TODO: Change to 0.1uF or 0.15uF cap \ndue to reduced current from the 10k pot"
-		(exclude_from_sim no)
-		(at 179.07 132.334 0)
-		(effects
-			(font
-				(size 1.27 1.27)
-			)
 		)
 	)
@@
 	(wire
 		(pts
-			(xy 120.65 73.66) (xy 154.94 73.66)
+			(xy 120.65 73.66) (xy 149.86 73.66)
 		)
 		(stroke
@@
 	(wire
 		(pts
-			(xy 143.51 86.36) (xy 143.51 90.17)
-		)
-		(stroke
-			(width 0)
-			(type default)
-		)
-	)
-	(wire
-		(pts
 			(xy 116.84 66.04) (xy 116.84 69.85)
 		)
@@
 	(wire
 		(pts
-			(xy 149.86 90.17) (xy 149.86 86.36)
+			(xy 154.94 83.82) (xy 154.94 90.17)
 		)
 		(stroke
@@
 	(wire
 		(pts
-			(xy 149.86 86.36) (xy 143.51 86.36)
+			(xy 154.94 83.82) (xy 161.29 83.82)
 		)
 		(stroke
@@
 	(wire
 		(pts
-			(xy 154.94 73.66) (xy 154.94 90.17)
+			(xy 149.86 73.66) (xy 149.86 90.17)
 		)
 		(stroke
@@
 			)
 		)
-		(property "Value" "10k_0603"
+		(property "Value" "100k_0603"
 			(at 218.44 97.79 90)
 			(effects
@@
 			)
 		)
-		(property "JLCPCB ID" "C25803"
+		(property "LCSC" "C25803"
 			(at 233.68 101.6 0)
 			(effects
@@
 		(unit 1)
 		(exclude_from_sim no)
-		(in_bom yes)
+		(in_bom no)
 		(on_board yes)
 		(dnp no)
@@
 			)
 		)
-		(property "Value" "10k_0603"
+		(property "Value" "1k_0603"
 			(at 224.79 110.49 90)
 			(effects
@@
 					(size 1.27 1.27)
 				)
-			)
-		)
-		(property "JLCPCB ID" "C25804"
-			(at 240.03 114.3 0)
-			(effects
-				(font
-					(size 1.27 1.27)
-				)
-				(hide yes)
 			)
 		)
@@
 			)
 		)
-		(property "Value" "100k"
+		(property "Value" "100k_0603"
 			(at 76.2 66.04 90)
 			(effects
@@
 			)
 		)
-		(property "JLCPCB ID" "C25803"
+		(property "LCSC" "C25803"
 			(at 91.44 62.23 0)
 			(effects
@@
 			)
 		)
-		(property "LCSC" "C6961"
-			(at 182.88 110.49 0)
-			(effects
-				(font
-					(size 1.27 1.27)
-				)
-				(hide yes)
-			)
-		)
 		(property "Manufacturer" "STMicroelectronics"
 			(at 182.88 110.49 0)
@@
 		)
 		(property "Part Number" "TL072CDT"
+			(at 182.88 110.49 0)
+			(effects
+				(font
+					(size 1.27 1.27)
+				)
+				(hide yes)
+			)
+		)
+		(property "LCSC" "C6961"
 			(at 182.88 110.49 0)
 			(effects
@@
 	)
 	(symbol
-		(lib_id "Isolator:NSL-32")
+		(lib_id "Lichen:NSL-32")
 		(at 152.4 97.79 270)
 		(unit 1)
 		(exclude_from_sim no)
-		(in_bom yes)
+		(in_bom no)
 		(on_board yes)
 		(dnp no)
@@
 			)
 		)
-		(property "LCSC" "C6961"
-			(at 92.71 66.04 0)
-			(effects
-				(font
-					(size 1.27 1.27)
-				)
-				(hide yes)
-			)
-		)
 		(property "Manufacturer" "STMicroelectronics"
 			(at 92.71 66.04 0)
@@
 		)
 		(property "Part Number" "TL072CDT"
+			(at 92.71 66.04 0)
+			(effects
+				(font
+					(size 1.27 1.27)
+				)
+				(hide yes)
+			)
+		)
+		(property "LCSC" "C6961"
 			(at 92.71 66.04 0)
 			(effects
@@
 			)
 		)
-		(property "Value" "100k"
+		(property "Value" "100k_0603"
 			(at 92.71 104.14 90)
 			(effects
@@
 			)
 		)
-		(property "JLCPCB ID" "C25803"
+		(property "LCSC" "C25803"
 			(at 107.95 107.95 0)
 			(effects
@@
 		(unit 1)
 		(exclude_from_sim no)
-		(in_bom yes)
+		(in_bom no)
 		(on_board yes)
 		(dnp no)
@@
 			)
 		)
-		(property "Footprint" "Lichen:Audio_Jack_Thonkiconn_Mono"
+		(property "Footprint" "Lichen:Audio_Jack_Thonkiconn_Mono_Right_Overhang"
 			(at 254.254 97.282 0)
 			(effects
@@
 	(symbol
 		(lib_id "power:GND")
-		(at 143.51 90.17 0)
+		(at 161.29 83.82 0)
+		(mirror y)
 		(unit 1)
 		(exclude_from_sim no)
@@
 		(fields_autoplaced yes)
 		(property "Reference" "#PWR030"
-			(at 143.51 96.52 0)
+			(at 161.29 90.17 0)
 			(effects
 				(font
@@
 		)
 		(property "Value" "GND"
-			(at 143.51 95.25 0)
+			(at 161.29 88.9 0)
 			(effects
 				(font
@@
 		)
 		(property "Footprint" ""
-			(at 143.51 90.17 0)
+			(at 161.29 83.82 0)
 			(effects
 				(font
@@
 		)
 		(property "Datasheet" ""
-			(at 143.51 90.17 0)
+			(at 161.29 83.82 0)
 			(effects
 				(font
@@
 		)
 		(property "Description" "Power symbol creates a global label with name \"GND\" , ground"
-			(at 143.51 90.17 0)
+			(at 161.29 83.82 0)
 			(effects
 				(font
@@
 			)
 		)
-		(property "Value" "100k"
+		(property "Value" "100k_0603"
 			(at 92.71 54.61 90)
 			(effects
@@
 			)
 		)
-		(property "JLCPCB ID" "C25803"
+		(property "LCSC" "C25803"
 			(at 107.95 58.42 0)
 			(effects
@@
 			)
 		)
-		(property "Value" "10k_0603"
+		(property "Value" "100k_0603"
 			(at 196.85 113.03 90)
 			(effects
@@
 			)
 		)
-		(property "JLCPCB ID" "C25803"
+		(property "LCSC" "C25803"
 			(at 212.09 109.22 0)
 			(effects
@@
 	)
 	(symbol
-		(lib_id "Lichen:Potentiometer")
+		(lib_id "Lichen:R_Potentiometer")
 		(at 116.84 73.66 0)
+		(mirror x)
 		(unit 1)
 		(exclude_from_sim no)
-		(in_bom yes)
+		(in_bom no)
 		(on_board yes)
 		(dnp no)
-		(fields_autoplaced yes)
 		(property "Reference" "RV2"
-			(at 114.3 72.3899 0)
+			(at 114.3 74.9301 0)
 			(effects
 				(font
@@
 		)
 		(property "Value" "B10K"
-			(at 114.3 74.9299 0)
+			(at 114.3 72.3901 0)
 			(effects
 				(font
@@
 		)
 		(property "Footprint" "Lichen:Potentiometer_Alpha_RD901_Eurorack"
-			(at 116.84 91.948 0)
+			(at 116.84 55.372 0)
 			(effects
 				(font
@@
 		)
 		(property "Datasheet" "https://www.thonk.co.uk/wp-content/uploads/2017/12/Alpha-9mm-Vertical-T18-RD901F-40-15K-B50K-0057.pdf"
-			(at 117.856 89.662 0)
+			(at 117.856 57.658 0)
 			(effects
 				(font
@@
 		)
 		(property "Description" "Alpha RD901 Vertical Snap-In Potentiometer"
-			(at 116.586 61.214 0)
+			(at 116.586 86.106 0)
 			(effects
 				(font
@@
 		)
 		(property "Part Number" "RD901F-40"
-			(at 116.84 87.63 0)
+			(at 116.84 59.69 0)
 			(effects
 				(font
@@
 		)
 		(property "Manufacturer" "Taiwan Alpha Electronic"
-			(at 117.348 85.598 0)
+			(at 117.348 61.722 0)
 			(effects
 				(font
@@
 		(unit 1)
 		(exclude_from_sim no)
-		(in_bom yes)
+		(in_bom no)
 		(on_board yes)
 		(dnp no)
@@
 			)
 		)
-		(property "Footprint" "Lichen:Audio_Jack_Thonkiconn_Mono"
+		(property "Footprint" "Lichen:Audio_Jack_Thonkiconn_Mono_Right_Overhang"
 			(at 42.926 47.752 0)
 			(effects
@@
 			)
 		)
-		(property "LCSC" "C6961"
-			(at 92.71 115.57 0)
-			(effects
-				(font
-					(size 1.27 1.27)
-				)
-				(hide yes)
-			)
-		)
 		(property "Manufacturer" "STMicroelectronics"
 			(at 92.71 115.57 0)
@@
 		)
 		(property "Part Number" "TL072CDT"
+			(at 92.71 115.57 0)
+			(effects
+				(font
+					(size 1.27 1.27)
+				)
+				(hide yes)
+			)
+		)
+		(property "LCSC" "C6961"
 			(at 92.71 115.57 0)
 			(effects
@@
 		(unit 1)
 		(exclude_from_sim no)
-		(in_bom yes)
+		(in_bom no)
 		(on_board yes)
 		(dnp no)
@@
 			)
 		)
-		(property "Footprint" "Lichen:Audio_Jack_Thonkiconn_Mono"
+		(property "Footprint" "Lichen:Audio_Jack_Thonkiconn_Mono_Right_Overhang"
 			(at 42.926 97.282 0)
 			(effects
@@
 			)
 		)
-		(property "Value" "100k"
+		(property "Value" "100k_0603"
 			(at 74.93 115.57 90)
 			(effects
@@
 			)
 		)
-		(property "JLCPCB ID" "C25803"
+		(property "LCSC" "C25803"
 			(at 90.17 111.76 0)
 			(effects
