File: Lichen_Design_Blocks.kicad_blocks/Eurorack Power - All JLC Basic.kicad_block/Eurorack Power - All JLC Basic.kicad_sch (KiCad schematic)
At the start: 7 parts

Commit message: Updates symbols, footprints, and design blocks.
Parts:
- removed C1, C2: 10uF_0805_25V, Lichen:C_0805, symbol Lichen:10uF_0805_50V
- removed D1, D2: Schottky, Diode_SMD:D_SMB_Handsoldering, symbol Lichen:Schottky_Diode
- added C15, C16, C27, C28, C29, C30: 10uF, Capacitor_SMD:C_1206_3216Metric, symbol Lichen:10uF_1206_50V
- added D7, D8: Schottky, Diode_SMD:D_SMA_Handsoldering, symbol Lichen:Schottky_Diode_JLC_Basic
- L1: Specifications 120Ω@100MHz 2A 50mΩ ±25% 0603 Ferrite Beads -> (none)
Connections:
- net +12V: now also C15.1, C16.1, C27.1, D7.1 (K)
- net -12V: now also C28.1, C29.1, C30.1, D8.2 (A)
- net GND: now also C15.2, C16.2, C27.2, C28.2, C29.2, C30.2
- net at L1.2: now also D7.2 (A)
- net at L2.2: now also D8.1 (K)
Other:
- note added: "Power circuit adapted from Paul Schreiber."
- note added: "The bulk capacitance is tripled here because these ceramic caps derate to 3.54V with an 11.9V DC bias (-64.6%). Schottkys diodes have been substituted with a JLC Basic part."
- note removed: "Power circuit from Paul Schreiber."
- moved on the sheet: L1, L2, PWR1
