File: lichen-baseline/Eurorack_Power.kicad_sch (KiCad schematic)
At the start: 11 parts

Commit message: Updates symbols, footprints, and design blocks.
Parts:
- L2: value 220Ω@100MHz -> 220R@100MHz
Changed lines of the file:
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@@
 			)
 		)
-		(property "Value" "220Ω@100MHz"
+		(property "Value" "220R@100MHz"
 			(at 137.16 63.754 90)
 			(effects
