File: lichen-crustose/lichen-crustose-processing-board/RingModulators.kicad_sch (KiCad schematic)
At the start: 12 parts

Commit message: Updates Lichen symbols and footprints. Fixes to Crustose and Vactrol VCA. Adds 3D model of the RP2350 dual USB board.
Connections:
- net GND: now also TR4.3, TR4.5; no longer TR4.2, TR4.4
- net RM_OUT_R: now also TR4.1; no longer TR4.6
- net at LED5.1 (K), LED8.2 (A): now also TR4.6; no longer TR4.1
- net at LED2.2 (A), LED6.1 (K): now also TR4.4; no longer TR4.3
Changed lines of the file:
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@@
 		(lib_id "Lichen:Transformer_42TM018")
 		(at 168.91 110.49 0)
+		(mirror y)
 		(unit 1)
 		(exclude_from_sim no)
