File: lichen-stereo-klein-filter/lichen-stereo-klein-filter-board/lichen-stereo-klein-filter-board.kicad_sch (KiCad schematic)
At the start: 85 parts, among them J8 Conn_02x07_Top_Bottom, U2 TL074, U3 TL074, U4 TL074, U5 TL074, U6 TL072

Commit message: feat: Updates Crustose, Cladonia and YouMe Transformer. Adds Stereo Latencies.
Parts:
- J8: value Conn_02x07_Top_Bottom -> 02x07 Pins; LCSC (none) -> C84004; Manufacturer (none) -> BOOMELE(Boom Precision Elec); Part Number (none) -> 2.54-2*7P针立贴
- R50, R8: symbol Lichen:13K_0603 -> Lichen:15K_0603; Display 13K -> 15K; JLCPCB ID C22797 -> (none); LCSC (none) -> C22809; Part Number 0603WAF1302T5E -> 0603WAF1502T5E
- R55, R56: JLCPCB ID C25804 -> (none); LCSC (none) -> C25804
- U2, U3, U4, U5: symbol Amplifier_Operational:TL074 -> Lichen:TL074; LCSC (none) -> C6964; Manufacturer (none) -> Texas Instruments; Part Number (none) -> TL074IDR
Connections:
- net AUDIO_OUT_UNFILTERED_L renamed AUDIO_OUT_DC_COUPLED_L
- net AUDIO_OUT_UNFILTERED_R renamed AUDIO_OUT_DC_COUPLED_R
Other:
- note added: "Just using up a couple of spare TL074 units?"
- moved on the sheet: R1, R54
