File: rp2350-dual-usb/Connectors.kicad_sch (KiCad schematic)
At the start: 22 parts, among them J2 USB_C_Receptacle_USB2.0_16P, J3 USB_C_Receptacle_USB2.0_14P, J4 TRS, J5 TRS, U3 USBLC6-2SC6, U4 USBLC6-2SC6, U5 HCPL-0631, U6 TPS25810RVC

Commit message: feat: Updates Crustose, Cladonia and YouMe Transformer. Adds Stereo Latencies.
Parts:
- C20: value 100nF_0402_16V -> 100nF
Changed lines of the file:
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@@
 		)
 		(instances
-			(project ""
+			(project "rp2350-dual-usb"
 				(path "/16ef7e10-64b2-4124-9408-fecb81ad1271/94926592-8b77-4efd-88ab-683ab0d2d180"
 					(reference "J5")
@@
 		)
 		(instances
-			(project ""
+			(project "rp2350-dual-usb"
 				(path "/16ef7e10-64b2-4124-9408-fecb81ad1271/94926592-8b77-4efd-88ab-683ab0d2d180"
 					(reference "C22")
@@
 		)
 		(instances
-			(project ""
+			(project "rp2350-dual-usb"
 				(path "/16ef7e10-64b2-4124-9408-fecb81ad1271/94926592-8b77-4efd-88ab-683ab0d2d180"
 					(reference "R19")
@@
 		)
 		(instances
-			(project ""
+			(project "rp2350-dual-usb"
 				(path "/16ef7e10-64b2-4124-9408-fecb81ad1271/94926592-8b77-4efd-88ab-683ab0d2d180"
 					(reference "U6")
@@
 		)
 		(instances
-			(project ""
+			(project "rp2350-dual-usb"
 				(path "/16ef7e10-64b2-4124-9408-fecb81ad1271/94926592-8b77-4efd-88ab-683ab0d2d180"
 					(reference "J4")
@@
 		)
 		(instances
-			(project ""
+			(project "rp2350-dual-usb"
 				(path "/16ef7e10-64b2-4124-9408-fecb81ad1271/94926592-8b77-4efd-88ab-683ab0d2d180"
 					(reference "C21")
@@
 		)
 		(instances
-			(project ""
+			(project "rp2350-dual-usb"
 				(path "/16ef7e10-64b2-4124-9408-fecb81ad1271/94926592-8b77-4efd-88ab-683ab0d2d180"
 					(reference "C23")
@@
 			)
 		)
-		(property "Value" "100nF_0402_16V"
+		(property "Value" "100nF"
 			(at 208.28 105.41 0)
 			(effects
@@
 		)
 		(instances
-			(project ""
+			(project "rp2350-dual-usb"
 				(path "/16ef7e10-64b2-4124-9408-fecb81ad1271/94926592-8b77-4efd-88ab-683ab0d2d180"
 					(reference "C20")
